File: hardware/amethyst.kicad_sch (KiCad schematic)
At the start: 43 parts, among them J2 USB_C_Receptacle_USB2.0_16P, SW86 SW_SPDT, U1 nRF52840, U2 BQ25185DLHR, Y1 Crystal_GND24_Small

Commit message: Routing complete
Parts:
- removed SW86: SW_SPDT, symbol Switch:SW_SPDT
- added L3: 4.7n, Inductor_SMD:L_0402_1005Metric, symbol Device:L
- added L4: 1,.8n, Inductor_SMD:L_0402_1005Metric, symbol Device:L
- added SW85: SW_SPST, Connector_PinHeader_1.00mm:PinHeader_1x02_P1.00mm_Vertical, symbol Switch:SW_SPST
- C24, C25: footprint (none) -> Capacitor_SMD:C_0402_1005Metric
- L2: footprint (none) -> Inductor_SMD:L_0402_1005Metric
Connections:
- net C1: now also U1.A20 (P1.10)
- net C2: now also U1.A16 (P1.13)
- net GND: now also L4.1
- net R4: now also U1.A14 (P1.15)
- net R5: now also U1.W24 (P1.02)
- net R6: now also U1.U24 (P1.04)
- net VSYS: now also SW85.2 (B)
- net at C20.1, C21.2, C22.2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: now also SW85.1 (A)
- net at C25.1, L2.1: now also L3.2, L4.2; no longer AE1.2 (PCB_Trace)
- new net: AE1.2 (PCB_Trace), L3.1
- no-connect marks 28 -> 27
Other:
- moved on the sheet: AE1

Commit message: Prod files
Parts:
- added H1, H2, H3, H4: MountingHole, MountingHole:MountingHole_3.2mm_M3, symbol Mechanical:MountingHole
- L4: value 1,.8n -> 1.8n
