File: hardware/amethyst.kicad_sch (KiCad schematic)
At the start: 49 parts, among them J2 USB_C_Receptacle_USB2.0_16P, SW85 SW_SPST, U1 nRF52840, U2 BQ25185DLHR, Y1 Crystal_GND24_Small

Commit message: new MCU
Parts:
- removed AE1: Antenna_Chip, RF_Antenna:Johanson_2450AT18x100, symbol Device:Antenna_Chip
- removed BT1: Battery_Cell, Connector_JST:JST_EH_B2B-EH-A_1x02_P2.50mm_Vertical, symbol Device:Battery_Cell
- removed C1, C2: C, Capacitor_SMD:C_0402_1005Metric, symbol Device:C
- removed C10: 100p, Capacitor_SMD:C_0402_1005Metric, symbol Device:C
- removed C11: 4.7u, Capacitor_SMD:C_0402_1005Metric, symbol Device:C
- removed C12, C21, C3, C7, C8, C9: 100n, Capacitor_SMD:C_0402_1005Metric, symbol Device:C
- removed D85, D86: LED, LED_SMD:LED_0402_1005Metric, symbol Device:LED
- removed L1: 10u, Inductor_SMD:L_smd_1212_3232metric, symbol Device:L
- removed L2, L3: 4.7n, Inductor_SMD:L_0402_1005Metric, symbol Device:L
- removed L4: 1.8n, Inductor_SMD:L_0402_1005Metric, symbol Device:L
- removed R3: 1k, Resistor_SMD:R_0402_1005Metric, symbol Device:R
- removed R4: 18k, Resistor_SMD:R_0402_1005Metric, symbol Device:R
- removed R5: 10k, Resistor_SMD:R_0402_1005Metric, symbol Device:R
- removed R6, R8: R, Resistor_SMD:R_0402_1005Metric, symbol Device:R
- removed SW85: SW_SPST, Connector_PinHeader_1.00mm:PinHeader_1x02_P1.00mm_Vertical, symbol Switch:SW_SPST
- removed U1: nRF52840, Package_DFN_QFN:Nordic_AQFN-73-1EP_7x7mm_P0.5mm, symbol MCU_Nordic:nRF52840
- removed U2: BQ25185DLHR, Package_DFN_QFN:Texas_DLH0010A_WSON-10-1EP_2.2x2mm_P0.4mm_EP0.9x1.5mm_ThermalVias, symbol easyeda2kicad:BQ25185DLHR
- removed Y1: Crystal_GND24_Small, Crystal:Crystal_SMD_3225-4Pin_3.2x2.5mm, symbol Device:Crystal_GND24_Small
- added C1, C2: 22p, Capacitor_SMD:C_0402_1005Metric, symbol Device:C_Small
- added R3, R6: 1k, Resistor_SMD:R_0402_1005Metric, symbol Device:R_Small
- added R4, R5: 27, Resistor_SMD:R_0402_1005Metric, symbol Device:R_Small
- added TP1, TP2: TestPoint, TestPoint:TestPoint_Pad_1.0x1.0mm, symbol Connector:TestPoint
- added U1: RP2040, Package_DFN_QFN:QFN-56-1EP_7x7mm_P0.4mm_EP3.2x3.2mm, symbol MCU_RaspberryPi:RP2040
- added U2: W25Q128JVS, Package_SO:SOIC-8_5.3x5.3mm_P1.27mm, symbol Memory_Flash:W25Q128JVS
- added U3: AMS1117-3.3, Package_TO_SOT_SMD:SOT-89-3, symbol Regulator_Linear:AMS1117-3.3
- added Y1: Crystal_GND24, Crystal:Crystal_SMD_3225-4Pin_3.2x2.5mm, symbol Device:Crystal_GND24
- C14, C23: value 1u -> 100n
- C15: value 47n -> 100n
- C18: value 850p -> 100n; now fitted; now in the parts list
- C20: value 10u -> 100n; footprint Capacitor_SMD:C_0805_2012Metric -> Capacitor_SMD:C_0402_1005Metric
- C22: value 1u -> 10u; footprint Capacitor_SMD:C_0402_1005Metric -> Capacitor_SMD:C_0805_2012Metric
- C24: value 0.8p -> 100n
- C25: value 0.5p -> 100n
- C5, C6: value 100n -> 1u
Connections:
- net DCC is gone; now on net +3V3: C14.2, C15.2
- net VSYS is gone; now on net +3V3: C16.2, C17.2
- net C1: now also U1.28 (GPIO17)
- net C10: now also U1.9 (GPIO7)
- net C11: now also U1.8 (GPIO6)
- net C12: now also U1.7 (GPIO5)
- net C13: now also U1.37 (GPIO25)
- net C14: now also U1.38 (GPIO26/ADC0)
- net C15: now also U1.39 (GPIO27/ADC1)
- net C16: now also U1.40 (GPIO28/ADC2)
- net C2: now also U1.30 (GPIO19)
- net C3: now also U1.32 (GPIO21)
- net C4: now also U1.34 (GPIO22)
- net C5: now also U1.6 (GPIO4)
- net C6: now also U1.5 (GPIO3)
- net C7: now also U1.4 (GPIO2)
- net C8: now also U1.3 (GPIO1)
- net C9: now also U1.2 (GPIO0)
- net D+: now also R5.1
- net D-: now also R4.1
- net GND: now also C20.1, C22.2, C24.1, C25.1, J2.S1 (SHIELD), C1.1, C2.1, TP2.1, U1.19 (TESTEN), U1.57 (GND), U2.4 (GND), U3.1 (GND), Y1.2 (G), Y1.4 (G); no longer C20.2, C22.1, C24.2, C25.2
- net R1: now also U1.41 (GPIO29/ADC3)
- net R2: now also U1.36 (GPIO24)
- net R3: now also U1.35 (GPIO23)
- net R4: now also U1.31 (GPIO20)
- net R5: now also U1.18 (GPIO15)
- net R6: now also U1.29 (GPIO18)
- net VBUS: now also U3.3 (VI)
- net +3V3: now reaches C19.2, C5.2
- net +3V3: now also C18.2, C20.2, C22.1, U1.1 (IOVDD), U1.10 (IOVDD), U1.22 (IOVDD), U1.26 (RUN), U1.33 (IOVDD), U1.42 (IOVDD), U1.43 (ADC_AVDD), U1.48 (USB_VDD), U1.49 (IOVDD), U2.8 (VCC), U3.2 (VO); no longer C6.2
- net +1V1: now reaches C23.2
- net +1V1: now also C24.2, C25.2, C6.2, U1.23 (DVDD), U1.45 (VREG_VOUT), U1.50 (DVDD)
- new net: R6.2, TP1.1
- new net: R5.2, U1.47 (USB_DP)
- new net: C2.2, R3.1, Y1.3
- new net: R4.2, U1.46 (USB_DM)
- new net: C1.2, U1.20 (XIN), Y1.1
- new net: R3.2, U1.21 (XOUT)
- new net QSPI_CLK: U1.52 (QSPI_SCLK), U2.6 (CLK)
- new net QSPI_CS: R6.1, U1.56 (~{QSPI_SS}), U2.1 (~{CS})
- new net QSPI_D0: U1.53 (QSPI_SD0), U2.5 (DI/IO_{0})
- new net QSPI_D1: U1.55 (QSPI_SD1), U2.2 (DO/IO_{1})
- new net QSPI_D2: U1.54 (QSPI_SD2), U2.3 (~{WP}/IO_{2})
- new net QSPI_D3: U1.51 (QSPI_SD3), U2.7 (~{HOLD}/~{RESET}/IO_{3})
- no-connect marks 27 -> 4
Other:
- note removed: "Status LED"
- note removed: "Switch(add footprint later)"

Commit message: PCB redone
Other:
- moved on the sheet: C1, C13, C14, C15, C16, C17, C18, C19, C2, C20, C22, C23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

Commit message: Latest Production files
Parts:
- C1, C2: value 22p -> 15p
Changed lines of the file:
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@@
 			)
 		)
-		(property "Value" "22p"
+		(property "Value" "15p"
 			(at 161.2963 214.63 90)
 			(show_name no)
@@
 			)
 		)
-		(property "Value" "22p"
+		(property "Value" "15p"
 			(at 161.2963 204.47 90)
 			(show_name no)
