File: hardware/matrix.kicad_sch (KiCad schematic)
At the start: 168 parts, among them SW1 SW_Push, SW10 SW_Push, SW11 SW_Push, SW12 SW_Push, SW13 SW_Push, SW14 SW_Push, SW15 SW_Push, SW16 SW_Push, SW17 SW_Push, SW18 SW_Push, SW19 SW_Push, SW2 SW_Push, SW20 SW_Push, SW21 SW_Push, SW22 SW_Push, SW23 SW_Push, SW24 SW_Push, SW25 SW_Push, SW26 SW_Push, SW27 SW_Push, SW28 SW_Push, SW29 SW_Push, SW3 SW_Push, SW30 SW_Push, SW31 SW_Push, SW32 SW_Push, SW33 SW_Push, SW34 SW_Push, SW35 SW_Push, SW36 SW_Push, SW37 SW_Push, SW38 SW_Push, SW39 SW_Push, SW4 SW_Push, SW40 SW_Push, SW41 SW_Push, SW42 SW_Push, SW43 SW_Push, SW44 SW_Push, SW45 SW_Push, SW46 SW_Push, SW47 SW_Push, SW48 SW_Push, SW49 SW_Push, SW5 SW_Push, SW50 SW_Push, SW51 SW_Push, SW52 SW_Push, SW53 SW_Push, SW54 SW_Push, SW55 SW_Push, SW56 SW_Push, SW57 SW_Push, SW58 SW_Push, SW59 SW_Push, SW6 SW_Push, SW60 SW_Push, SW61 SW_Push, SW62 SW_Push, SW63 SW_Push, SW64 SW_Push, SW65 SW_Push, SW66 SW_Push, SW67 SW_Push, SW68 SW_Push, SW69 SW_Push, SW7 SW_Push, SW70 SW_Push, SW71 SW_Push, SW72 SW_Push, SW73 SW_Push, SW74 SW_Push, SW75 SW_Push, SW76 SW_Push, SW77 SW_Push, SW78 SW_Push, SW79 SW_Push, SW8 SW_Push, SW80 SW_Push, SW81 SW_Push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

Commit message: Layout done
Parts:
- SW1, SW10, SW11, SW12, SW13, SW14, SW15, SW16, SW17, SW18, SW19, SW2, SW20, SW21, SW22, SW23, SW24, SW25, SW26, SW27, SW28, SW29, SW3, SW31, SW33, SW34, SW35, SW36, SW37, SW38, SW39, SW4, SW40, SW41, SW42, SW43, SW44, SW46, SW48, SW49, SW5, SW50, SW51, SW52, SW53, SW54, SW55, SW56, SW57, SW58, SW6, SW60, SW62, SW63, SW64, SW65, SW66, SW67, SW68, SW69, SW7, SW70, SW71, SW73, SW74, SW79, SW8, SW80, SW81, SW82, SW83, SW84, SW9: footprint (none) -> Button_Switch_Keyboard:SW_Cherry_MX_1.00u_PCB
- SW30: footprint (none) -> Button_Switch_Keyboard:SW_Cherry_MX_2.00u_PCB
- SW32, SW45: footprint (none) -> Button_Switch_Keyboard:SW_Cherry_MX_1.50u_PCB
- SW47, SW72: footprint (none) -> Button_Switch_Keyboard:SW_Cherry_MX_1.75u_PCB
- SW59, SW61: footprint (none) -> Button_Switch_Keyboard:SW_Cherry_MX_2.25u_PCB
- SW75, SW76, SW77: footprint (none) -> Button_Switch_Keyboard:SW_Cherry_MX_1.25u_PCB
- SW78: footprint (none) -> Button_Switch_Keyboard:SW_Cherry_MX_6.25u_PCB

Commit message: PCB Routing
Connections:
- net C10: now also SW79.1
- net C11: now also SW80.1; no longer SW79.1
- net C12: now also SW81.1; no longer SW80.1
- net C13: no longer SW81.1
- net C6: now also SW78.1
- net C7: no longer SW78.1
Other:
- moved on the sheet: D78, D79, D80, D81, SW78, SW79, SW80, SW81
