File: hardware/amethyst.kicad_pcb (KiCad board)
At the start: 2 copper layers, 323.3 x 119 mm, 213 parts, among them J2 USB_C_Receptacle_USB2.0_16P, SW1 SW_Push, SW10 SW_Push, SW11 SW_Push, SW12 SW_Push, SW13 SW_Push, SW14 SW_Push, SW15 SW_Push, SW16 SW_Push, SW17 SW_Push, SW18 SW_Push, SW19 SW_Push, SW2 SW_Push, SW20 SW_Push, SW21 SW_Push, SW22 SW_Push, SW23 SW_Push, SW24 SW_Push, SW25 SW_Push, SW26 SW_Push, SW27 SW_Push, SW28 SW_Push, SW29 SW_Push, SW3 SW_Push, SW30 SW_Push, SW31 SW_Push, SW32 SW_Push, SW33 SW_Push, SW34 SW_Push, SW35 SW_Push, SW36 SW_Push, SW37 SW_Push, SW38 SW_Push, SW39 SW_Push, SW4 SW_Push, SW40 SW_Push, SW41 SW_Push, SW42 SW_Push, SW43 SW_Push, SW44 SW_Push, SW45 SW_Push, SW46 SW_Push, SW47 SW_Push, SW48 SW_Push, SW49 SW_Push, SW5 SW_Push, SW50 SW_Push, SW51 SW_Push, SW52 SW_Push, SW53 SW_Push, SW54 SW_Push, SW55 SW_Push, SW56 SW_Push, SW57 SW_Push, SW58 SW_Push, SW59 SW_Push, SW6 SW_Push, SW60 SW_Push, SW61 SW_Push, SW62 SW_Push, SW63 SW_Push, SW64 SW_Push, SW65 SW_Push, SW66 SW_Push, SW67 SW_Push, SW68 SW_Push, SW69 SW_Push, SW7 SW_Push, SW70 SW_Push, SW71 SW_Push, SW72 SW_Push, SW73 SW_Push, SW74 SW_Push, SW75 SW_Push, SW76 SW_Push, SW77 SW_Push, SW78 SW_Push, SW79 SW_Push, SW8 SW_Push, SW80 SW_Push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

Commit message: Prod files
Parts:
- added G***: LOGO, LOGO, F.Cu at (222.8, 157.7)
- added G***: LOGO, LOGO, B.Cu at (351.7, 56.5)
- added H1: MountingHole, MountingHole:MountingHole_3.2mm_M3, F.Cu at (102.8, 137.0)
- added H2: MountingHole, MountingHole:MountingHole_3.2mm_M3, F.Cu at (83.1, 71.9)
- added H3: MountingHole, MountingHole:MountingHole_3.2mm_M3, F.Cu at (312.2, 72.5)
- added H4: MountingHole, MountingHole:MountingHole_3.2mm_M3, F.Cu at (328.3, 138.4)
- L4: value 1,.8n -> 1.8n

Commit message: new MCU
Parts:
- removed AE1: Antenna_Chip, RF_Antenna:Johanson_2450AT18x100
- removed BT1: Battery_Cell, Connector_JST:JST_EH_B2B-EH-A_1x02_P2.50mm_Vertical
- removed C10: 100p, Capacitor_SMD:C_0402_1005Metric
- removed C11: 4.7u, Capacitor_SMD:C_0402_1005Metric
- removed C12, C21, C3, C7, C8, C9: 100n, Capacitor_SMD:C_0402_1005Metric
- removed D85, D86: LED, LED_SMD:LED_0402_1005Metric
- removed L1: 10u, Inductor_SMD:L_smd_1212_3232metric
- removed L2, L3: 4.7n, Inductor_SMD:L_0402_1005Metric
- removed L4: 1.8n, Inductor_SMD:L_0402_1005Metric
- removed R8: R, Resistor_SMD:R_0402_1005Metric
- removed SW85: SW_SPST, Connector_PinHeader_1.00mm:PinHeader_1x02_P1.00mm_Vertical
- added TP1: TestPoint, TestPoint:TestPoint_Pad_1.0x1.0mm, B.Cu at (378.4, 62.8)
- added TP2: TestPoint, TestPoint:TestPoint_Pad_1.0x1.0mm, B.Cu at (376.4, 62.8)
- added U3: AMS1117-3.3, Package_TO_SOT_SMD:SOT-89-3, B.Cu at (369.3, 62.4)
- C1, C2: value C -> 22p
- C14, C23: value 1u -> 100n
- C15: value 47n -> 100n
- C18: value 850p -> 100n
- C20: value 10u -> 100n; footprint Capacitor_SMD:C_0805_2012Metric -> Capacitor_SMD:C_0402_1005Metric
- C22: value 1u -> 10u; footprint Capacitor_SMD:C_0402_1005Metric -> Capacitor_SMD:C_0805_2012Metric
- C24: value 0.8p -> 100n
- C25: value 0.5p -> 100n
- C5, C6: value 100n -> 1u
- R4: value 18k -> 27
- R5: value 10k -> 27
- R6: value R -> 1k
- U1: value nRF52840 -> RP2040; footprint Package_DFN_QFN:Nordic_AQFN-73-1EP_7x7mm_P0.5mm -> Package_DFN_QFN:QFN-56-1EP_7x7mm_P0.4mm_EP3.2x3.2mm
- U2: value BQ25185DLHR -> W25Q128JVS; footprint Package_DFN_QFN:Texas_DLH0010A_WSON-10-1EP_2.2x2mm_P0.4mm_EP0.9x1.5mm_ThermalVias -> Package_SO:SOIC-8_5.3x5.3mm_P1.27mm
- Y1: value Crystal_GND24_Small -> Crystal_GND24
- moved R3 20.2 mm to (371.8, 82.0), turned to 0 degrees
- moved C23 19.6 mm to (368.6, 83.7), turned to 0 degrees
- moved R6 14.1 mm to (380.3, 63.8), turned to 90 degrees
- moved C20 13.1 mm to (377.7, 73.4)
- moved C15 13.1 mm to (366.4, 70.3), turned to -90 degrees
- moved C25 12.5 mm to (368.3, 70.5)
- moved C19 10.8 mm to (369.0, 82.7), turned to 0 degrees
- moved C24 10.5 mm to (367.4, 70.5), turned to -90 degrees
- moved C14 9.52 mm to (369.0, 81.8), turned to 0 degrees
- moved C4 9.35 mm to (376.1, 58.6), turned to 180 degrees
- moved U2 8.12 mm to (376.9, 67.9), turned to 180 degrees
- moved C16 8.11 mm to (366.0, 73.5)
- moved C17 8.10 mm to (366.0, 72.6)
- moved C5 7.68 mm to (366.0, 71.7), turned to 0 degrees
- moved R4 7.19 mm to (369.3, 68.9), turned to -90 degrees
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Connections:
- C1 pad 2: Net-(U1-XC1) -> Net-(U1-XIN)
- C14 pad 2: /DCC -> +3V3
- C15 pad 2: /DCC -> +3V3
- C16 pad 2: /VSYS -> +3V3
- C17 pad 2: /VSYS -> +3V3
- C18 pad 2: Net-(U1-DEC5) -> +3V3
- C19 pad 2: Net-(C19-Pad2) -> +3V3
- C2 pad 2: Net-(U1-XC2) -> Net-(C2-Pad2)
- C20 pad 1: Net-(SW85-A) -> GND
- C20 pad 2: GND -> +3V3
- C22 pad 1: GND -> +3V3
- C22 pad 2: Net-(SW85-A) -> GND
- C23 pad 2: Net-(BT1-+) -> +1V1
- C24 pad 1: Net-(U1-ANT) -> GND
- C24 pad 2: GND -> +1V1
- C25 pad 1: Net-(C25-Pad1) -> GND
- C25 pad 2: GND -> +1V1
- C5 pad 2: Net-(C19-Pad2) -> +3V3
- C6 pad 2: Net-(C19-Pad2) -> +1V1
- R3 pad 1: Net-(U2-ISET) -> Net-(C2-Pad2)
- R3 pad 2: GND -> Net-(U1-XOUT)
- R4 pad 1: Net-(U2-ILIM/VSET) -> D-
- R4 pad 2: GND -> Net-(U1-USB_DM)
- R5 pad 1: Net-(U2-TS/MR) -> D+
- R5 pad 2: GND -> Net-(U1-USB_DP)
- R6 pad 1: Net-(D85-A) -> /QSPI_CS
- R6 pad 2: /VSYS -> Net-(R6-Pad2)
- U2 pad 1: Net-(SW85-A) -> /QSPI_CS
- U2 pad 2: Net-(BT1-+) -> /QSPI_D1
- U2 pad 3: Net-(D85-K) -> /QSPI_D2
- U2 pad 5: GND -> /QSPI_D0
- U2 pad 6: Net-(U2-TS/MR) -> /QSPI_CLK
- U2 pad 7: Net-(U2-ILIM/VSET) -> /QSPI_D3
- U2 pad 8: Net-(U2-ISET) -> +3V3
- Y1 pad 1: Net-(U1-XC1) -> Net-(U1-XIN)
- Y1 pad 3: Net-(U1-XC2) -> Net-(C2-Pad2)
Routing:
- net +3V3: track 0.00 -> 87.4 mm, vias 0 -> 7
- net Net-(C19-Pad2): track 37.7 -> 0.00 mm, vias 5 -> 0
- net GND: track 44.6 -> 9.98 mm, vias 40 -> 35
- net Net-(BT1-+): track 29.5 -> 0.00 mm, vias 1 -> 0
- net +1V1: track 0.00 -> 29.0 mm, vias 0 -> 5
- net VBUS: track 28.3 -> 9.78 mm, vias 2 -> 0
- net R6: track 394.9 -> 378.3 mm
- net R5: track 365.3 -> 349.8 mm
- net /QSPI_CS: track 0.00 -> 15.3 mm
- net /DCC: track 14.1 -> 0.00 mm, vias 2 -> 0
- net /VSYS: track 12.2 -> 0.00 mm, vias 2 -> 0
- net C10: track 259.4 -> 271.5 mm
- net /QSPI_D1: track 0.00 -> 12.0 mm
- net C11: track 239.5 -> 251.0 mm
- net C12: track 215.2 -> 226.0 mm
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- removed copper zone on B.Cu, net /VSYS
- removed copper zone on B.Cu, net Net-(SW85-A)
Other:
- board size 323.3 x 119 mm -> 321.3 x 119 mm
- board text added: "BOOT GND"

Commit message: PCB redone
Routing:
- net VBUS: track 9.78 -> 16.7 mm
- net D+: track 12.5 -> 15.0 mm
- net D-: track 12.5 -> 14.4 mm
- net +3V3: track 87.4 -> 88.3 mm
- net GND: vias 35 -> 36
