File: hardware/amethyst.kicad_pcb (KiCad board)
At the start: 2 copper layers, 321.3 x 119 mm, 204 parts, among them J2 USB_C_Receptacle_USB2.0_16P, SW1 SW_Push, SW10 SW_Push, SW11 SW_Push, SW12 SW_Push, SW13 SW_Push, SW14 SW_Push, SW15 SW_Push, SW16 SW_Push, SW17 SW_Push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

Commit message: Latest Production files
Parts:
- C1, C2: value 22p -> 15p
